File: PCBs/Full-Board_rev1/3v3_Regulator.kicad_sch (KiCad schematic)
At the start: 6 parts, among them Q1 TPS630250RNCT

Commit message: added ESP32 peripherals
Parts:
- R1, R2: symbol Device:R -> Device:R_Small_US
Changed lines of the file:
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@@
+	)
+	(junction
+		(at 99.06 76.2)
+		(diameter 0)
+		(color 0 0 0 0)
+	)
+	(junction
+		(at 177.8 76.2)
+		(diameter 0)
+		(color 0 0 0 0)
+	)
+	(junction
+		(at 115.57 76.2)
+		(diameter 0)
+		(color 0 0 0 0)
+	)
+	(junction
+		(at 195.58 76.2)
+		(diameter 0)
+		(color 0 0 0 0)
+	)
+	(junction
+		(at 115.57 83.82)
+		(diameter 0)
+		(color 0 0 0 0)
 	)
 	(junction
@@
 		(color 0 0 0 0)
 	)
-	(junction
-		(at 99.06 76.2)
-		(diameter 0)
-		(color 0 0 0 0)
-	)
-	(junction
-		(at 115.57 76.2)
-		(diameter 0)
-		(color 0 0 0 0)
-	)
-	(junction
-		(at 195.58 76.2)
-		(diameter 0)
-		(color 0 0 0 0)
-	)
-	(junction
-		(at 115.57 83.82)
-		(diameter 0)
-		(color 0 0 0 0)
-	)
-	(junction
-		(at 177.8 76.2)
-		(diameter 0)
-		(color 0 0 0 0)
-	)
 	(wire
 		(pts
@@
 	(wire
 		(pts
+			(xy 161.29 104.14) (xy 168.91 104.14)
+		)
+		(stroke
+			(width 0)
+			(type default)
+		)
+	)
+	(wire
+		(pts
+			(xy 195.58 87.63) (xy 195.58 91.44)
+		)
+		(stroke
+			(width 0)
+			(type default)
+		)
+	)
+	(wire
+		(pts
 			(xy 177.8 76.2) (xy 195.58 76.2)
 		)
@@
 	(wire
 		(pts
-			(xy 161.29 104.14) (xy 168.91 104.14)
-		)
-		(stroke
-			(width 0)
-			(type default)
-		)
-	)
-	(wire
-		(pts
-			(xy 195.58 87.63) (xy 195.58 91.44)
-		)
-		(stroke
-			(width 0)
-			(type default)
-		)
-	)
-	(wire
-		(pts
 			(xy 115.57 88.9) (xy 115.57 83.82)
 		)
@@
 	(wire
 		(pts
+			(xy 177.8 83.82) (xy 177.8 85.09)
+		)
+		(stroke
+			(width 0)
+			(type default)
+		)
+	)
+	(wire
+		(pts
 			(xy 195.58 76.2) (xy 205.74 76.2)
 		)
@@
 	(wire
 		(pts
+			(xy 177.8 76.2) (xy 177.8 77.47)
+		)
+		(stroke
+			(width 0)
+			(type default)
+		)
+	)
+	(wire
+		(pts
 			(xy 161.29 83.82) (xy 177.8 83.82)
 		)
@@
 	(wire
 		(pts
+			(xy 177.8 82.55) (xy 177.8 83.82)
+		)
+		(stroke
+			(width 0)
+			(type default)
+		)
+	)
+	(wire
+		(pts
 			(xy 195.58 76.2) (xy 195.58 80.01)
+		)
+		(stroke
+			(width 0)
+			(type default)
+		)
+	)
+	(wire
+		(pts
+			(xy 177.8 90.17) (xy 177.8 91.44)
 		)
 		(stroke
@@
 	)
 	(symbol
-		(lib_id "Device:R")
+		(lib_id "Device:R_Small_US")
 		(at 177.8 87.63 0)
 		(unit 1)
@@
 		)
 		(property "Footprint" ""
-			(at 176.022 87.63 90)
+			(at 177.8 87.63 0)
 			(effects
 				(font
@@
 			)
 		)
-		(property "Description" "Resistor"
+		(property "Description" "Resistor, small US symbol"
 			(at 177.8 87.63 0)
 			(effects
@@
 	)
 	(symbol
-		(lib_id "Device:R")
+		(lib_id "Device:R_Small_US")
 		(at 177.8 80.01 0)
 		(unit 1)
@@
 		)
 		(property "Footprint" ""
-			(at 176.022 80.01 90)
+			(at 177.8 80.01 0)
 			(effects
 				(font
@@
 			)
 		)
-		(property "Description" "Resistor"
+		(property "Description" "Resistor, small US symbol"
 			(at 177.8 80.01 0)
 			(effects

Commit message: Fixed some rules checker errors
Connections:
- no-connect marks 0 -> 4
Changed lines of the file:
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@@
 		(color 0 0 0 0)
 	)
+	(no_connect
+		(at 120.65 81.28)
+	)
+	(no_connect
+		(at 166.37 78.74)
+	)
+	(no_connect
+		(at 166.37 81.28)
+	)
+	(no_connect
+		(at 120.65 78.74)
+	)
 	(wire
 		(pts
@@
 	(wire
 		(pts
+			(xy 120.65 78.74) (xy 125.73 78.74)
+		)
+		(stroke
+			(width 0)
+			(type default)
+		)
+	)
+	(wire
+		(pts
+			(xy 120.65 81.28) (xy 125.73 81.28)
+		)
+		(stroke
+			(width 0)
+			(type default)
+		)
+	)
+	(wire
+		(pts
 			(xy 161.29 104.14) (xy 168.91 104.14)
 		)
@@
 	(wire
 		(pts
+			(xy 161.29 78.74) (xy 166.37 78.74)
+		)
+		(stroke
+			(width 0)
+			(type default)
+		)
+	)
+	(wire
+		(pts
 			(xy 177.8 83.82) (xy 177.8 85.09)
 		)
@@
 		)
 		(stroke
+			(width 0)
+			(type default)
+		)
+	)
+	(wire
+		(pts
+			(xy 161.29 81.28) (xy 166.37 81.28)
+		)
+		(stroke
