File: PCBs/Full-Board_rev1/Full-Board_rev1.kicad_sch (KiCad schematic)
At the start: 25 parts, among them J10 Conn_01x11, J11 Conn_01x02_Pin, J12 Conn_01x02, J13 Conn_01x04, J2 Conn_01x05, J3 Conn_01x05, J4 Conn_01x05, J5 Conn_01x05, J6 MotorWithEncoder_M2, J7 MotorWithEncoder_M1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

Commit message: make sure everything is saved and pushed
Connections:
- net ENC_PH_B_M2 is gone; now on net 3V3: J6.3 (Pin_3), Q2.16 (GPIO18)
- net 3V3: no longer J6.4 (Pin_4), J7.4 (Pin_4)
- new net Status_LED/3V3: J6.4 (Pin_4), J7.4 (Pin_4)
Other:
- note removed: "Motor Drivers"
- note removed: "Motors w/ Encoders"
- moved on the sheet: C1, C2, C5, C6, C?, D1, J10, J11, J12, J13, J2, J3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
