File: PCBs/Power-Board_rev1/Power-Board_rev1.kicad_sch (KiCad schematic)
At the start: 7 parts, among them J1 Conn_01x04, Q1 RT6150AGQW

Commit message: Power Board Schematic
Parts:
- added C3: 10uF, Capacitor_SMD:C_0805_2012Metric_Pad1.18x1.45mm_HandSolder, symbol Device:C_Small
- C1: footprint (none) -> Capacitor_SMD:C_0805_2012Metric_Pad1.18x1.45mm_HandSolder; JLCPCB Part# (none) -> C95841
- C2: value 20uF -> 10uF; footprint (none) -> Capacitor_SMD:C_0805_2012Metric_Pad1.18x1.45mm_HandSolder; JLCPCB Part# (none) -> C531341
- J1: footprint (none) -> Connector:FanPinHeader_1x04_P2.54mm_Vertical; now left out of the parts list
- L1: footprint (none) -> Inductor_SMD:L_Changjiang_FTC252012S
- Q1: JLCPCB Part# (none) -> C147971
- R1: footprint (none) -> Resistor_SMD:R_0603_1608Metric_Pad0.98x0.95mm_HandSolder; JLCPCB Part# (none) -> C23183
- R2: footprint (none) -> Resistor_SMD:R_0603_1608Metric_Pad0.98x0.95mm_HandSolder; JLCPCB Part# (none) -> C23121
Connections:
- net GND: now also C3.2
- net VOUT: now also C3.1
Other:
- moved on the sheet: C1, C2, J1, L1, Q1, R1, R2

Commit message: updated power board layout, added extra pads for additional capacitors
Parts:
- added C4, C5: 10uF, Capacitor_SMD:C_0805_2012Metric_Pad1.18x1.45mm_HandSolder, symbol Device:C_Small
- J1: footprint Connector:FanPinHeader_1x04_P2.54mm_Vertical -> Connector_PinHeader_2.54mm:PinHeader_1x04_P2.54mm_Vertical
Connections:
- net GND: now also C4.2, C5.2
- net VIN: now also C4.1
- net VOUT: now also C5.1
Other:
- title: (none) -> Power Board
- moved on the sheet: J1

Commit message: Power board layout rev-1 mostly finished
Parts:
- C2, C3, C5: JLCPCB Part# C531341 -> C95841
- J1: footprint Connector_PinHeader_2.54mm:PinHeader_1x04_P2.54mm_Vertical -> Header:PinHeader_1x04_P2.54mm_Vertical_GND2
- L1: JLCPCB Part# (none) -> C5832372
